File: Hardware/Tom Titor Rebuild/Tom Titor Logic Board Rebuilt.sch (EAGLE design)
At the start: 38 parts, among them J2 KLDX-0202-B, SW1 FSMRA4JH, SW2 FSMRA4JH, SW3 102-1261-EV, U1 LM7805CT, U2 1364-HVPS-H, U3 PIC16F628A, U4 DS1307+, U5 DS3232SN, X1 CRYSTAL, X2 32.768kHz

Commit message: Library mismatch fix
Major errors involved with a late change that was made to the component library. Don't let your layout and schematic get out of sync kids.
Parts:
- C1: value 33μF -> 33µF; device My Imported Components:E-CAPS_US -> My Imported Components:CPOL-USE2-5
- C2: device My Imported Components:E-CAPS_USE3.5-8 -> My Imported Components:CPOL-USE3.5-8
- C3, C4, C5, C6: device My Imported Components:FK18X7R1H104K -> My Imported Components:C-US
- F1: device My Imported Components:5X20MM_FUSE -> My Imported Components:FUSE
- J1: device My Imported Components:FE08-1 -> My Imported Components:FE08
- J3: device My Imported Components:MA06-1 -> My Imported Components:MA06
- NC1, NC2, NC3: device My Imported Components:FE02-1 -> My Imported Components:FE02
- R1, R2, R3, R31, R32, R4, R6: device My Imported Components:R-US_0207/10 -> My Imported Components:R-US0207/10
