File: Hardware/Tom Titor Rebuild/Tom Titor Nixie Board Rebuilt.sch (EAGLE design)
At the start: 42 parts, among them J4 1, T0 IN-14, T1 IN-14, T2 IN-14, T3 IN-14, T4 IN-14, T5 IN-14, T6 IN-14, T7 IN-14, U6 HV5622PG-G, U7 HV5622PG-G, U8 HV5622PG-G

Commit message: Library mismatch fix
Major errors involved with a late change that was made to the component library. Don't let your layout and schematic get out of sync kids.
Parts:
- R10, R11, R12, R13, R14, R15, R16, R17, R18, R19, R20, R21, R22, R23, R24, R25, R26, R27, R28, R29, R30, R7, R8, R9: device My Imported Components:R-US_0207/10 -> My Imported Components:R-US0207/10
